Commit message: updates for simulation

File: src/bumperbot_description/urdf/bumperbot.urdf.xacro (robot description, xacro)
@@ -1,4 +1,6 @@
  <robot xmlns:xacro="http://www.ros.org/wiki/xacro" name="bumperbot">
     <xacro:include filename="inertial_macros.xacro"/>
+    <xacro:include filename="bumperbot_gazebo.xacro" />
+    <xacro:include filename="bumperbot_ros2_control.xacro" />
     <link name="base_footprint" />
     <link name="base_link">

File: src/bumperbot_description/urdf/bumperbot_gazebo.xacro (robot description, xacro)
@@ -1,4 +1,18 @@
 <?xml version="1.0" ?>
 <robot name="bumperbot" xmlns:xacro="http://www.ros.org/wiki/xacro">
+    <transmission name="wheel_right_transmission">
+        <plugin>transmission_interface/SimpleTransmission</plugin>
+        <actuator name="wheel_right_motor" role="actuator_right" />
+        <joint name="wheel_right_joint" role="joint_right">
+            <mechanical_reduction>1.0</mechanical_reduction>
+        </joint>
+    </transmission>
+    <transmission name="wheel_left_transmission">
+        <plugin>transmission_interface/SimpleTransmission</plugin>
+        <actuator name="wheel_left_motor" role="actuator_left" />
+        <joint name="wheel_left_joint" role="joint_left">
+            <mechanical_reduction>1.0</mechanical_reduction>
+        </joint>
+    </transmission>
     <gazebo reference="wheel_right_link">
         <mu1>100000000000000.0</mu1>
@@ -9,4 +23,5 @@
         <maxVel>0.1</maxVel>
         <fdir1>1 0 0</fdir1>
+        <material>Gazebo/Red</material>
     </gazebo>
     <gazebo reference="wheel_left_link">
@@ -18,4 +33,5 @@
         <maxVel>0.1</maxVel>
         <fdir1>1 0 0</fdir1>
+        <material>Gazebo/Red</material>
     </gazebo>
     <gazebo reference="caster_front_link">
@@ -35,3 +51,10 @@
         <maxVel>0.1</maxVel>
     </gazebo>
+    <gazebo>
+        <plugin filename="libgazebo_ros2_control.so" name="gazebo_ros2_control">
+            <robot_param>robot_description</robot_param>
+            <robot_param_node>robot_state_publisher</robot_param_node>
+            <parameters>$(find bumperbot_controller)/config/bumperbot_controllerss.yaml</parameters>
+        </plugin>
+    </gazebo>
 </robot>
